Commit message: last changes before second RAS submission

File: robot_descriptions/climbingrobot_description/urdf/climb_wall2.xacro (robot description, xacro)
@@ -20,7 +20,10 @@
 <xacro:arg name="anchorZ" default="10."/>
 <xacro:arg name="wall_inclination" default="0.0"/>
-<xacro:arg name="obstacle_x" default="-0.5"/>
-<xacro:arg name="obstacle_y" default="2.5"/>
-<xacro:arg name="obstacle_z" default="-6"/>
+<xacro:arg name="obstacle_location_x" default="-0.5"/>
+<xacro:arg name="obstacle_location_y" default="2.5"/>
+<xacro:arg name="obstacle_location_z" default="-6"/>
+<xacro:arg name="obstacle_size_x" default="1.5"/>
+<xacro:arg name="obstacle_size_y" default="1.5"/>
+<xacro:arg name="obstacle_size_z" default="0.866"/>
 	<link name="wall">
 		<inertial>
@@ -29,5 +32,5 @@
   	     </inertial>
 		<visual > <!-- dont put name otherwise gazebo discards color-->
- 			<origin xyz="${$(arg anchorZ)/2 *sin($(arg wall_inclination))}  0 ${$(arg anchorZ)/2}" rpy="0  -$(arg wall_inclination) 0"/>
+ 			<origin xyz="${$(arg anchorZ)/2 *sin($(arg wall_inclination))}  0 ${$(arg anchorZ) * (1-0.5*cos($(arg wall_inclination)))}" rpy="0  -$(arg wall_inclination) 0"/>
 			<geometry>
 				<box size="0.1 $(arg anchorZ) $(arg anchorZ)"/>
@@ -36,5 +39,5 @@
 		</visual>
 	        <collision name="box">
-		       <origin xyz="${$(arg anchorZ)/2 *sin($(arg wall_inclination))} 0 ${$(arg anchorZ)/2}" rpy="0  -$(arg wall_inclination) 0"/>
+		       <origin xyz="${$(arg anchorZ)/2 *sin($(arg wall_inclination))} 0 ${$(arg anchorZ) * (1-0.5*cos($(arg wall_inclination)))}" rpy="0  -$(arg wall_inclination) 0"/>
 		       <geometry>
  				<box size="0.1 $(arg anchorZ) $(arg anchorZ)"/>
@@ -74,14 +77,14 @@
   	        </inertial>
 		<visual > <!-- dont put name otherwise gazebo discards color-->
- 			  <origin rpy="0 0 0" xyz="$(arg obstacle_x) $(arg obstacle_y)  ${$(arg anchorZ) + $(arg obstacle_z)} "/>
+ 			  <origin rpy="0 0 0" xyz="$(arg obstacle_location_x) $(arg obstacle_location_y)  ${$(arg anchorZ) + $(arg obstacle_location_z)} "/>
 			<geometry>
-	                  <mesh filename="package://climbingrobot_description/meshes/ellipsoid.stl" scale="1 1 1"/>
+	                  <mesh filename="package://climbingrobot_description/meshes/ellipsoid.stl" scale="${$(arg obstacle_size_x)/1.5}  ${$(arg obstacle_size_y)/1.5}  ${$(arg obstacle_size_z)/0.866} "/>
 	                </geometry>
 			 <material name="orange"/>
 		</visual>
 		<collision>
-			<origin rpy="0 0 0" xyz="$(arg obstacle_x) $(arg obstacle_y)  ${$(arg anchorZ) + $(arg obstacle_z)} "/>
+			<origin rpy="0 0 0" xyz="$(arg obstacle_location_x) $(arg obstacle_location_y)  ${$(arg anchorZ) + $(arg obstacle_location_z)} "/>
 			 <geometry>
-	                  <mesh filename="package://climbingrobot_description/meshes/ellipsoid.stl" scale="1 1 1"/>
+	                  <mesh filename="package://climbingrobot_description/meshes/ellipsoid.stl" scale="${$(arg obstacle_size_x)/1.5}  ${$(arg obstacle_size_y)/1.5}  ${$(arg obstacle_size_z)/0.866} "/>
 	                </geometry>
 	       </collision>

File: robot_descriptions/climbingrobot_description/urdf/climbingrobot2.xacro (robot description, xacro)
@@ -13,4 +13,5 @@
    <xacro:arg name="hoist_distance" default="0.1"/>
    <xacro:arg name="hoist_base_distanceZ" default="0.05"/>
+   <xacro:arg name="double_propeller" default="false"/>
     <xacro:include filename="$(find climbingrobot_description)/gazebo/gazebo.urdf.xacro">
         <xacro:arg name="task_period" value="$(arg task_period)"/>
@@ -195,5 +196,5 @@
   <!-- Anchor 2   -->
    <joint name="anchor2_position" type="fixed">
-        <origin rpy="0 0 0" xyz="0 $(arg anchor2Y) 0"/>
+        <origin rpy="0 0 0" xyz="0 ${$(arg anchor2Y)-$(arg anchorY)} 0"/>
         <parent link="anchor"/>
         <child link="anchor_2"/>
@@ -567,6 +568,11 @@
   <!-- END LOWER LEG LINK -->
   <!-- Joint between the base and the ${prefix} upper leg -->
+   <xacro:unless value="$(arg double_propeller)">
+   	<xacro:include filename="$(find climbingrobot_description)/urdf/propellers.urdf.xacro"/>
+   </xacro:unless>
+   <xacro:if value="$(arg double_propeller)">
+         <xacro:include filename="$(find climbingrobot_description)/urdf/propellers_couple.urdf.xacro"/>
+   </xacro:if>
    <xacro:include filename="$(find climbingrobot_description)/urdf/gazebo.urdf.xacro"/>
-   <xacro:include filename="$(find climbingrobot_description)/urdf/propellers.urdf.xacro"/>
    <xacro:climbingrobot_transmission/>
 </robot>

File: robot_descriptions/climbingrobot_description/urdf/climbingrobot2landing.xacro (robot description, xacro)
@@ -14,4 +14,5 @@
    <xacro:arg name="hoist_base_distanceZ" default="0.05"/>
    <xacro:arg name="lowerleg_landing_length" default="0.3"/>
+    <xacro:arg name="double_propeller" default="false"/>
     <xacro:property name="WHEEL_pos" value="0.10183" />
     <xacro:include filename="$(find climbingrobot_description)/gazebo/gazebo.urdf.xacro">
@@ -197,5 +198,5 @@
   <!-- Anchor 2   -->
    <joint name="anchor2_position" type="fixed">
-        <origin rpy="0 0 0" xyz="0 $(arg anchor2Y) 0"/>
+        <origin rpy="0 0 0" xyz="0 ${$(arg anchor2Y)-$(arg anchorY)} 0"/>
         <parent link="anchor"/>
         <child link="anchor_2"/>
@@ -603,6 +604,6 @@
                <inertial>
                     <origin xyz="0 0 0" rpy="0 0 0"/>
-                    <mass value="0.00693606"/>
-                    <inertia ixx="0.00000057" ixy="0.0" ixz="0.0" iyy="0.00000084" iyz="0.0" izz="0.00000053"/>
+                    <mass value="0.5"/>
+                   <inertia ixx="0.00001" ixy="0.0" ixz="0.0" iyy="0.00001" iyz="0.0" izz="0.00001"/>
                 </inertial>
         </link>
@@ -636,6 +637,6 @@
                <inertial>
                     <origin xyz="0 0 0" rpy="0 0 0"/>
-                    <mass value="0.00693606"/>
-                    <inertia ixx="0.00000057" ixy="0.0" ixz="0.0" iyy="0.00000084" iyz="0.0" izz="0.00000053"/>
+                    <mass value="0.5"/>
+                    <inertia ixx="0.00001" ixy="0.0" ixz="0.0" iyy="0.00001" iyz="0.0" izz="0.00001"/>
                 </inertial>
         </link>
@@ -815,4 +816,10 @@
   <!-- Joint between the base and the ${prefix} upper leg -->
    <xacro:include filename="$(find climbingrobot_description)/urdf/gazebo.urdf.xacro"/>
+   <xacro:unless value="$(arg double_propeller)">
+   	<xacro:include filename="$(find climbingrobot_description)/urdf/propellers.urdf.xacro"/>
+   </xacro:unless>
+   <xacro:if value="$(arg double_propeller)">
+         <xacro:include filename="$(find climbingrobot_description)/urdf/propellers_couple.urdf.xacro"/>
+   </xacro:if>
    <xacro:climbingrobot_transmission/>
 </robot>

File: robot_descriptions/climbingrobot_description/urdf/climbingrobot2landing_paper.xacro (robot description, xacro)
@@ -197,5 +197,5 @@
   <!-- Anchor 2   -->
    <joint name="anchor2_position" type="fixed">
-        <origin rpy="0 0 0" xyz="0 $(arg anchor2Y) 0"/>
+        <origin rpy="0 0 0" xyz="0 ${$(arg anchor2Y)-$(arg anchorY)} 0"/>
         <parent link="anchor"/>
         <child link="anchor_2"/>

File: robot_descriptions/climbingrobot_description/urdf/propellers.urdf.xacro (robot description, xacro)
@@ -1,10 +1,10 @@
 <?xml version="1.0"?>
 <robot xmlns:xacro="http://ros.org/wiki/xacro">
-  <joint name="propeller_sx_location" type="fixed">
+  <joint name="propeller_location" type="fixed">
     <parent link="base_link"/>
-    <child link="propeller_sx"/>
-    <origin rpy="0 -1.57 0" xyz="0.07 -0.05  0.025"/>
+    <child link="propeller"/>
+    <origin rpy="0 -1.57 0" xyz="0.07 0  0.025"/>
   </joint>
-  <link name="propeller_sx">
+  <link name="propeller">
     <visual>
       <origin rpy="0 0 0" xyz="0 0 0"/>
@@ -17,19 +17,3 @@
     </visual>
   </link>
-  <joint name="propeller_dx_location" type="fixed">
-    <parent link="base_link"/>
-    <child link="propeller_dx"/>
-    <origin rpy="0 -1.57 0" xyz="0.07 0.05 0.025"/>
-  </joint>
-  <link name="propeller_dx">
-    <visual>
-      <origin rpy="0 0 0" xyz="0 0 0"/>
-      <geometry>
-        <mesh filename="package://climbingrobot_description/meshes/propeller_simple.stl" scale="0.002 0.002 0.002"/>
-      </geometry>
-	<material name="blue">
-        <color rgba="0 1 0 1.0"/>
-      </material>
-    </visual>
-  </link>
 </robot>
