Commit message: commit for multi-jump

File: robot_descriptions/climbingrobot_description/urdf/climbingrobot2landing_paper.xacro (robot description, xacro)
@@ -440,4 +440,14 @@
       <inertia ixx="0.00000057" ixy="0.0" ixz="0.0" iyy="0.00000084" iyz="0.0" izz="0.00000053"/>
     </inertial>
+    <!-- FOOT VISUAL -->
+    <visual>
+      <origin rpy="0 0 0" xyz="0 0 0"/>
+      <geometry>
+        <sphere radius="0.02175" />
+      </geometry>
+	<material name="black">
+		<color rgba="0.263 0.298 0.369 1"/>
+	</material>
+    </visual>
     <!-- FOOT COLLISION -->
     <collision>
@@ -519,4 +529,14 @@
       <inertia ixx="0.00000057" ixy="0.0" ixz="0.0" iyy="0.00000084" iyz="0.0" izz="0.00000053"/>
     </inertial>
+    <!-- FOOT VISUAL -->
+    <visual>
+      <origin rpy="0 0 0" xyz="0 0 0"/>
+      <geometry>
+        <sphere radius="0.02175" />
+      </geometry>
+	<material name="black">
+		<color rgba="0.263 0.298 0.369 1"/>
+	</material>
+    </visual>
     <!-- FOOT COLLISION -->
     <collision>

File: robot_urdf/generated_urdf/climbingrobot2.urdf (robot description, URDF)
Before this commit: robot climbingrobot2, 21 links, 20 joints
Links:
- removed link propeller_dx
- removed link propeller_sx
- added link propeller; visual mesh filename=package://climbingrobot_description/meshes/propeller_simple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 scale=0.002 0.002 0.002
Joints:
- removed joint propeller_dx_location
- removed joint propeller_sx_location
- added joint propeller_location: type fixed, parent base_link, child propeller, origin xyz=0.07 0  0.025 rpy=0 -1.57 0
