Commit message: last massive cleanup

File: robot_descriptions/climbingrobot_description/urdf/climbingrobot2.xacro (robot description, xacro)
@@ -338,13 +338,13 @@
   <joint name="wire_base_yaw_r" type="revolute">
     <parent link="pre-base3_2"/>
-    <child link="fake_link"/>
+    <child link="fake_link_end_of_right_rope"/>
     <limit effort="1000" velocity="100.0" lower="-100" upper="100"/>
     <!-- joint rotates about x axis -->
     <axis xyz="0 0 1"/>
-    <origin rpy="0 0 0" xyz="0.0 0.0 0.0"/>
-    <!-- pybullet simulation parameters -->
-    <dynamics damping="0.0" friction="0.0"/>
-  </joint>
-  <link name="fake_link">
+     <origin  xyz="0 ${-$(arg hoist_distance)/2} ${-$(arg hoist_base_distanceZ)}" rpy="0 0 0" />
+    <!-- pybullet simulation parameters -->
+    <dynamics damping="0.0" friction="0.0"/>
+  </joint>
+  <link name="fake_link_end_of_right_rope">
     <inertial>
       <origin rpy="0 0 0" xyz="0 0 0.0"/>
@@ -356,6 +356,6 @@
  <gazebo>
 	  <joint name="fixed_joint" type="fixed">
-		 <pose>0 ${$(arg hoist_distance)/2} $(arg hoist_base_distanceZ) 0 0 0 0</pose>
-		 <parent>fake_link</parent>
+		 <pose>0 0 0 0 0 0 0</pose>
+		 <parent>fake_link_end_of_right_rope</parent>
 		 <child>base_link</child>
 	  </joint>
